File: PicoFraise/PicoFraiseJST/PicoFraise.kicad_sch (KiCad schematic)
At the start: 21 parts, among them J1 Conn_01x06, J2 Conn_01x06, J3 Conn_01x06, J4 Conn_01x06, J5 Conn_01x06, J6 Conn_01x06, J7 Reset, J8 12-24V input, U1 Pico, U2 L7805

Commit message: update PicoFraiseJST
Parts:
- added D2: 100mA, Diode_SMD:D_SMA, symbol Device:D_Schottky
- J8: footprint TerminalBlock:TerminalBlock_bornier-2_P5.08mm -> TerminalBlock:TerminalBlock_bornier-3_P5.08mm; symbol Connector:Conn_01x02_Socket -> Connector:Conn_01x03_Socket
Connections:
- net +5V: now also J8.3 (Pin_3)
- net RX: now also D2.2 (A)
- net TX: now also D2.1 (K)
Changed lines of the file:
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@@
+    (stroke (width 0) (type default))
+  )
+  (wire (pts (xy 200.66 124.46) (xy 198.12 124.46))
     (stroke (width 0) (type default))
   )
@@
     (stroke (width 0) (type default))
   )
+  (wire (pts (xy 170.18 115.57) (xy 198.12 115.57))
+    (stroke (width 0) (type default))
+  )
   (wire (pts (xy 88.9 62.23) (xy 88.9 64.77))
     (stroke (width 0) (type default))
@@
     (stroke (width 0) (type default))
   )
+  (wire (pts (xy 198.12 115.57) (xy 198.12 124.46))
+    (stroke (width 0) (type default))
+  )
   (wire (pts (xy 148.59 77.47) (xy 132.08 77.47))
     (stroke (width 0) (type default))
@@
   )
   (wire (pts (xy 135.89 87.63) (xy 132.08 87.63))
+    (stroke (width 0) (type default))
+  )
+  (wire (pts (xy 170.18 121.92) (xy 170.18 115.57))
     (stroke (width 0) (type default))
   )
@@
   (label "RX" (at 231.14 59.69 180) (fields_autoplaced)
     (effects (font (size 1.27 1.27)) (justify right bottom))
+  )
+  (label "RX" (at 193.04 60.96 180) (fields_autoplaced)
+    (effects (font (size 1.27 1.27)) (justify right bottom))
+  )
+  (label "TX" (at 200.66 60.96 0) (fields_autoplaced)
+    (effects (font (size 1.27 1.27)) (justify left bottom))
   )
   (label "RX" (at 132.08 92.71 0) (fields_autoplaced)
@@
     )
   )
-  (symbol (lib_id "Connector:Conn_01x02_Socket") (at 165.1 127 180) (unit 1)
+  (symbol (lib_id "Connector:Conn_01x03_Socket") (at 165.1 124.46 180) (unit 1)
     (in_bom yes) (on_board yes) (dnp no)
     (property "Reference" "J8" (at 163.83 127 0)
@@
       (effects (font (size 1.27 1.27)) (justify left))
     )
-    (property "Footprint" "TerminalBlock:TerminalBlock_bornier-2_P5.08mm" (at 165.1 127 0)
-      (effects (font (size 1.27 1.27)) hide)
-    )
-    (property "Datasheet" "~" (at 165.1 127 0)
-      (effects (font (size 1.27 1.27)) hide)
-    )
-    (pin "2")
-    (pin "1")
+    (property "Footprint" "TerminalBlock:TerminalBlock_bornier-3_P5.08mm" (at 165.1 124.46 0)
+      (effects (font (size 1.27 1.27)) hide)
+    )
+    (property "Datasheet" "~" (at 165.1 124.46 0)
+      (effects (font (size 1.27 1.27)) hide)
+    )
+    (pin "2")
+    (pin "1")
+    (pin "3")
     (instances
       (project "PicoFraise"
@@
     )
   )
-  (symbol (lib_id "power:+5V") (at 198.12 124.46 0) (unit 1)
-    (in_bom yes) (on_board yes) (dnp no)
-    (property "Reference" "#PWR026" (at 198.12 128.27 0)
-      (effects (font (size 1.27 1.27)) hide)
-    )
-    (property "Value" "+5V" (at 198.12 120.65 0)
-      (effects (font (size 1.27 1.27)))
-    )
-    (property "Footprint" "" (at 198.12 124.46 0)
-      (effects (font (size 1.27 1.27)) hide)
-    )
-    (property "Datasheet" "" (at 198.12 124.46 0)
+  (symbol (lib_id "power:+5V") (at 200.66 124.46 0) (unit 1)
+    (in_bom yes) (on_board yes) (dnp no)
+    (property "Reference" "#PWR026" (at 200.66 128.27 0)
+      (effects (font (size 1.27 1.27)) hide)
+    )
+    (property "Value" "+5V" (at 200.66 120.65 0)
+      (effects (font (size 1.27 1.27)))
+    )
+    (property "Footprint" "" (at 200.66 124.46 0)
+      (effects (font (size 1.27 1.27)) hide)
+    )
+    (property "Datasheet" "" (at 200.66 124.46 0)
       (effects (font (size 1.27 1.27)) hide)
     )
@@
     )
   )
+  (symbol (lib_id "Device:D_Schottky") (at 196.85 60.96 180) (unit 1)
+    (in_bom yes) (on_board yes) (dnp no)
+    (property "Reference" "D2" (at 196.85 55.88 0)
+      (effects (font (size 1.27 1.27)))
+    )
+    (property "Value" "100mA" (at 196.85 58.42 0)
+      (effects (font (size 1.27 1.27)))
+    )
+    (property "Footprint" "Diode_SMD:D_SMA" (at 196.85 60.96 0)
+      (effects (font (size 1.27 1.27)) hide)
+    )
+    (property "Datasheet" "~" (at 196.85 60.96 0)
+      (effects (font (size 1.27 1.27)) hide)
+    )
+    (pin "1")
+    (pin "2")
+    (instances
+      (project "PicoFraise"
+        (path "/24107a89-373f-4f98-9004-7e880608beb2"
+          (reference "D2") (unit 1)
+        )
+      )
+    )
+  )
   (symbol (lib_id "power:GND") (at 96.52 100.33 270) (unit 1)
     (in_bom yes) (on_board yes) (dnp no) (fields_autoplaced)
@@
   (symbol (lib_id "Device:D_Schottky") (at 173.99 124.46 180) (unit 1)
     (in_bom yes) (on_board yes) (dnp no)
-    (property "Reference" "D1" (at 173.99 120.65 0)
-      (effects (font (size 1.27 1.27)))
-    )
-    (property "Value" "1A" (at 171.45 121.92 0)
-      (effects (font (size 1.27 1.27)))
-    )
+    (property "Reference" "D1" (at 173.99 119.38 0)
+      (effects (font (size 1.27 1.27)))
+    )
+    (property "Value" "1A" (at 173.99 121.92 0)
+      (effects (font (size 1.27 1.27)))
+    )
